Commit message: Updated launch file for non-demo mode and added random values as test

File: kuka_arm/urdf/target.urdf.xacro (robot description, xacro)
@@ -22,5 +22,5 @@
   </link>
   <gazebo reference="target_link_1">
-    <material>Gazebo/Blue</material>
+    <material>Gazebo/Green</material>
     <mu1>1.0</mu1>
     <mu2>1.0</mu2>

Commit message: Changed Material to TieDyed

File: kuka_arm/urdf/target.urdf.xacro (robot description, xacro)
@@ -22,5 +22,5 @@
   </link>
   <gazebo reference="target_link_1">
-    <material>Gazebo/Green</material>
+    <material>Gazebo/TieDyed</material>
     <mu1>1.0</mu1>
     <mu2>1.0</mu2>

Commit message: Rotated Target to face forward on load.

File: kuka_arm/urdf/target.urdf.xacro (robot description, xacro)
@@ -7,5 +7,5 @@
     </inertial>
     <visual>
-      <origin xyz="0 0 0"/>
+      <origin xyz="0 0 0" rpy="0 0 -1.57"/>
       <geometry>
         <cylinder radius="0.05" length="0.25"/>
